File: hardware/hardware.kicad_sch (KiCad schematic)
At the start: 1 part, among them U1 XC6SLX4-CPG196

Commit message: restart hardware proj
Parts:
- removed U1: XC6SLX4-CPG196, symbol FPGA_Xilinx_Spartan6:XC6SLX4-CPG196
Other:
- note removed: "All input voltages shall be <= 3.9V (shoot for 3.3)"
- note removed: "https://docs.amd.com/v/u/en-US/ds162 VCCint is ~1.2V max VCCaux is ~3.3V max https://docs.amd.com/v/u/en-US/ug393 - Design guide for Spartan 6"

Commit message: jdafklafkldj
Parts:
- added U1: XC6SLX4-CPG196, symbol FPGA_Xilinx_Spartan6:XC6SLX4-CPG196
Other:
- note added: "All input voltages shall be <= 3.9V (shoot for 3.3)"
- note added: "https://docs.amd.com/v/u/en-US/ds162 VCCint is ~1.2V max VCCaux is ~3.3V max https://docs.amd.com/v/u/en-US/ug393 - Design guide for Spartan 6"
