File: hardware/hardware.kicad_sch (KiCad schematic)
At the start: 2 parts

Commit message: update level shifter adapter board schematic
Parts:
- added J1, J2, J3, J4: Conn_01x10_Socket, Connector_PinSocket_2.54mm:PinSocket_1x10_P2.54mm_Vertical, symbol Connector:Conn_01x10_Socket
- added J5, J6, J7, J8: Conn_01x10_Pin, Connector_PinHeader_2.54mm:PinHeader_1x10_P2.54mm_Vertical, symbol Connector:Conn_01x10_Pin
- added R10, R2, R3, R4, R5, R6, R7, R8, R9: 10k, Resistor_SMD:R_0402_1005Metric_Pad0.72x0.64mm_HandSolder, symbol Device:R_Small
- added U10, U2, U3, U4, U5, U6, U7, U8, U9: ~, hardware:NXB0104_XQFN12, symbol custom_symbols:NXB0104_XQFN12
- R1: footprint (none) -> Resistor_SMD:R_0402_1005Metric_Pad0.72x0.64mm_HandSolder
- U1: footprint (none) -> hardware:NXB0104_XQFN12
Connections:
- net +3V3: now also J2.1 (Pin_1), R10.1, R2.1, R3.1, R4.1, R5.1, R6.1, R7.1, R8.1, R9.1, U10.1 (VCC_A), U2.1 (VCC_A), U3.1 (VCC_A), U4.1 (VCC_A), U5.1 (VCC_A), U6.1 (VCC_A), U7.1 (VCC_A), U8.1 (VCC_A), U9.1 (VCC_A)
- net +5V: now also J6.1 (Pin_1), U10.14 (VCC_B), U2.14 (VCC_B), U3.14 (VCC_B), U4.14 (VCC_B), U5.14 (VCC_B), U6.14 (VCC_B), U7.14 (VCC_B), U8.14 (VCC_B), U9.14 (VCC_B)
- net GND: now also J7.9 (Pin_9), U10.7 (GND), U2.7 (GND), U3.7 (GND), U4.7 (GND), U5.7 (GND), U6.7 (GND), U7.7 (GND), U8.7 (GND), U9.7 (GND)
- net A14_5V: now reaches U1.10 (B4)
- net A14_5V: now also J5.4 (Pin_4)
- net A13_5V: now reaches U1.11 (B3)
- net A13_5V: now also J5.3 (Pin_3)
- net A12_5V: now reaches U1.12 (B2)
- net A12_5V: now also J5.2 (Pin_2)
- net A11_5V: now reaches U1.13 (B1)
- net A11_5V: now also J5.1 (Pin_1)
- net A11_FPGA: now reaches U1.2 (A1)
- net A11_FPGA: now also J1.1 (Pin_1)
- net A12_FPGA: now reaches U1.3 (A2)
- net A12_FPGA: now also J1.2 (Pin_2)
- net A13_FPGA: now reaches U1.4 (A3)
- net A13_FPGA: now also J1.3 (Pin_3)
- net A14_FPGA: now reaches U1.5 (A4)
- net A14_FPGA: now also J1.4 (Pin_4)
- new net: R2.2, U2.8 (OE)
- new net: R10.2, U10.8 (OE)
- new net: R9.2, U9.8 (OE)
- new net: R4.2, U4.8 (OE)
- new net: R7.2, U7.8 (OE)
- new net: R6.2, U6.8 (OE)
- new net: R5.2, U5.8 (OE)
- new net: R8.2, U8.8 (OE)
- new net: R3.2, U3.8 (OE)
- new net A0_5V: J7.10 (Pin_10), U8.12 (B2)
- new net A0_FPGA: J4.10 (Pin_10), U8.3 (A2)
- new net A10_5V: J8.10 (Pin_10), U10.10 (B4)
- new net A10_FPGA: J3.10 (Pin_10), U10.5 (A4)
- new net A15_5V: J5.5 (Pin_5), U2.13 (B1)
- new net A15_FPGA: J1.5 (Pin_5), U2.2 (A1)
- new net A1_5V: J8.1 (Pin_1), U8.11 (B3)
- new net A1_FPGA: J3.1 (Pin_1), U8.4 (A3)
- new net A2_5V: J8.2 (Pin_2), U8.10 (B4)
- new net A2_FPGA: J3.2 (Pin_2), U8.5 (A4)
- new net A3_5V: J8.3 (Pin_3), U9.13 (B1)
- new net A3_FPGA: J3.3 (Pin_3), U9.2 (A1)
- new net A4_5V: J8.4 (Pin_4), U9.12 (B2)
- new net A4_FPGA: J3.4 (Pin_4), U9.3 (A2)
- new net A5_5V: J8.5 (Pin_5), U9.11 (B3)
- new net A5_FPGA: J3.5 (Pin_5), U9.4 (A3)
- new net A6_5V: J8.6 (Pin_6), U9.10 (B4)
- new net A6_FPGA: J3.6 (Pin_6), U9.5 (A4)
- new net A7_5V: J8.7 (Pin_7), U10.13 (B1)
- new net A7_FPGA: J3.7 (Pin_7), U10.2 (A1)
- new net A8_5V: J8.8 (Pin_8), U10.12 (B2)
- new net A8_FPGA: J3.8 (Pin_8), U10.3 (A2)
- new net A9_5V: J8.9 (Pin_9), U10.11 (B3)
- new net A9_FPGA: J3.9 (Pin_9), U10.4 (A3)
- new net BUSAK_5V: J7.3 (Pin_3), U6.11 (B3)
- new net BUSAK_FPGA: J4.3 (Pin_3), U6.4 (A3)
- new net BUSRQ_5V: J7.5 (Pin_5), U7.13 (B1)
- new net BUSRQ_FPGA: J4.5 (Pin_5), U7.2 (A1)
- new net CLK: J1.6 (Pin_6), U2.3 (A2)
- new net CLK_5V: J5.6 (Pin_6), U2.12 (B2)
- new net D0_5V: J6.4 (Pin_4), U4.12 (B2)
- new net D0_FPGA: J2.4 (Pin_4), U4.3 (A2)
- new net D1_5V: J6.5 (Pin_5), U4.11 (B3)
- new net D1_FPGA: J2.5 (Pin_5), U4.4 (A3)
- new net D2_5V: J6.2 (Pin_2), U3.10 (B4)
- new net D2_FPGA: J2.2 (Pin_2), U3.5 (A4)
- new net D3_5V: J5.8 (Pin_8), U2.10 (B4)
- new net D3_FPGA: J1.8 (Pin_8), U2.5 (A4)
- new net D4_5V: J5.7 (Pin_7), U2.11 (B3)
- new net D4_FPGA: J1.7 (Pin_7), U2.4 (A3)
- new net D5_5V: J5.9 (Pin_9), U3.13 (B1)
- new net D5_FPGA: J1.9 (Pin_9), U3.2 (A1)
- new net D6_5V: J5.10 (Pin_10), U3.12 (B2)
- new net D6_FPGA: J1.10 (Pin_10), U3.3 (A2)
- new net D7_5V: J6.3 (Pin_3), U4.13 (B1)
- new net D7_FPGA: J2.3 (Pin_3), U4.2 (A1)
- new net HALT_5V: J6.8 (Pin_8), U5.12 (B2)
- new net HALT_FPGA: J2.8 (Pin_8), U5.3 (A2)
- new net INT_5V: J6.6 (Pin_6), U4.10 (B4)
- new net INT_FPGA: J2.6 (Pin_6), U4.5 (A4)
- new net IORQ_5V: J6.10 (Pin_10), U5.10 (B4)
- new net IORQ_FPGA: J2.10 (Pin_10), U5.5 (A4)
- new net M1_5V: J7.7 (Pin_7), U7.11 (B3)
- new net M1_FPGA: J4.7 (Pin_7), U7.4 (A3)
- new net MREQ_5V: J6.9 (Pin_9), U5.11 (B3)
- new net MREQ_FPGA: J2.9 (Pin_9), U5.4 (A3)
- new net NMI_5V: J6.7 (Pin_7), U5.13 (B1)
- new net NMI_FPGA: J2.7 (Pin_7), U5.2 (A1)
- new net RD_5V: J7.1 (Pin_1), U6.13 (B1)
- new net RD_FPGA: J4.1 (Pin_1), U6.2 (A1)
- new net RESET_5V: J7.6 (Pin_6), U7.12 (B2)
- new net RESET_FPGA: J4.6 (Pin_6), U7.3 (A2)
- new net RFSH_5V: J7.8 (Pin_8), U7.10 (B4)
- new net RFSH_FPGA: J4.8 (Pin_8), U7.5 (A4)
- new net WAIT_5V: J7.4 (Pin_4), U6.10 (B4)
- new net WAIT_FPGA: J4.4 (Pin_4), U6.5 (A4)
- new net WR_5V: J7.2 (Pin_2), U6.12 (B2)
- new net WR_FPGA: J4.2 (Pin_2), U6.3 (A2)
- no-connect marks 0 -> 5
Other:
- note added: "Connectors for side 1"
- note added: "Connectors for side 2"
- note added: "Lets use this single pin from the FPGA and always tie it high to 3V3 to power the level shifters."
- note added: "Pins 1-20 (ascending order)"
- note added: "Pins 21-40 (ascending order)"
- note added: "This A1 --> is GND on original Z80"
- note added: "This A3 --> is VCC (5V) on original Z80"
- note added: "https://www.retrocompute.co.uk/zilog-z80-pinout/ This is the PHYSICAL PINOUT"
- moved on the sheet: R1, U1

Commit message: first general schematic/layout pushed. need to look into some stuff
Parts:
- R1, R10, R2, R3, R4, R5, R6, R7, R8, R9: footprint Resistor_SMD:R_0402_1005Metric_Pad0.72x0.64mm_HandSolder -> Resistor_SMD:R_0201_0603Metric
Connections:
- net +5V: now also U1.12 (VCC_B), U10.12 (VCC_B), U2.12 (VCC_B), U3.12 (VCC_B), U4.12 (VCC_B), U5.12 (VCC_B), U6.12 (VCC_B), U7.12 (VCC_B), U8.12 (VCC_B), U9.12 (VCC_B); no longer U1.14 (VCC_B), U10.14 (VCC_B), U2.14 (VCC_B), U3.14 (VCC_B), U4.14 (VCC_B), U5.14 (VCC_B), U6.14 (VCC_B), U7.14 (VCC_B), U8.14 (VCC_B), U9.14 (VCC_B)
- net A0_5V: now also U8.10 (B2); no longer U8.12 (B2)
- net A10_5V: now also U6.8 (B4); no longer U10.10 (B4)
- net A10_FPGA: now also U6.5 (A4); no longer U10.5 (A4)
- net A11_5V: now also U1.11 (B1); no longer U1.13 (B1)
- net A12_5V: now also U1.10 (B2); no longer U1.12 (B2)
- net A13_5V: now also U1.9 (B3); no longer U1.11 (B3)
- net A14_5V: now also U1.8 (B4); no longer U1.10 (B4)
- net A15_5V: now also U2.11 (B1); no longer U2.13 (B1)
- net A1_5V: now also U8.9 (B3); no longer U8.11 (B3)
- net A2_5V: now also U8.8 (B4); no longer U8.10 (B4)
- net A3_5V: now also U7.11 (B1); no longer U9.13 (B1)
- net A3_FPGA: now also U7.2 (A1); no longer U9.2 (A1)
- net A4_5V: now also U7.10 (B2); no longer U9.12 (B2)
- net A4_FPGA: now also U7.3 (A2); no longer U9.3 (A2)
- net A5_5V: now also U7.9 (B3); no longer U9.11 (B3)
- net A5_FPGA: now also U7.4 (A3); no longer U9.4 (A3)
- net A6_5V: now also U7.8 (B4); no longer U9.10 (B4)
- net A6_FPGA: now also U7.5 (A4); no longer U9.5 (A4)
- net A7_5V: now also U6.11 (B1); no longer U10.13 (B1)
- net A7_FPGA: now also U6.2 (A1); no longer U10.2 (A1)
- net A8_5V: now also U6.10 (B2); no longer U10.12 (B2)
- net A8_FPGA: now also U6.3 (A2); no longer U10.3 (A2)
- net A9_5V: now also U6.9 (B3); no longer U10.11 (B3)
- net A9_FPGA: now also U6.4 (A3); no longer U10.4 (A3)
- net BUSAK_5V: now also U10.9 (B3); no longer U6.11 (B3)
- net BUSAK_FPGA: now also U10.4 (A3); no longer U6.4 (A3)
- net BUSRQ_5V: now also U9.11 (B1); no longer U7.13 (B1)
- net BUSRQ_FPGA: now also U9.2 (A1); no longer U7.2 (A1)
- net CLK_5V: now also U2.10 (B2); no longer U2.12 (B2)
- net D0_5V: now also U4.10 (B2); no longer U4.12 (B2)
- net D1_5V: now also U4.9 (B3); no longer U4.11 (B3)
- net D2_5V: now also U3.8 (B4); no longer U3.10 (B4)
- net D3_5V: now also U2.8 (B4); no longer U2.10 (B4)
- net D4_5V: now also U2.9 (B3); no longer U2.11 (B3)
- net D5_5V: now also U3.11 (B1); no longer U3.13 (B1)
- net D6_5V: now also U3.10 (B2); no longer U3.12 (B2)
- net D7_5V: now also U4.11 (B1); no longer U4.13 (B1)
- net GND: now also U1.6 (GND), U10.6 (GND), U2.6 (GND), U3.6 (GND), U4.6 (GND), U5.6 (GND), U6.6 (GND), U7.6 (GND), U8.6 (GND), U9.6 (GND); no longer U1.7 (GND), U10.7 (GND), U2.7 (GND), U3.7 (GND), U4.7 (GND), U5.7 (GND), U6.7 (GND), U7.7 (GND), U8.7 (GND), U9.7 (GND)
- net HALT_5V: now also U5.10 (B2); no longer U5.12 (B2)
- net INT_5V: now also U4.8 (B4); no longer U4.10 (B4)
- net IORQ_5V: now also U5.8 (B4); no longer U5.10 (B4)
- net M1_5V: now also U9.9 (B3); no longer U7.11 (B3)
- net M1_FPGA: now also U9.4 (A3); no longer U7.4 (A3)
- net MREQ_5V: now also U5.9 (B3); no longer U5.11 (B3)
- net NMI_5V: now also U5.11 (B1); no longer U5.13 (B1)
- net RD_5V: now also U10.11 (B1); no longer U6.13 (B1)
- net RD_FPGA: now also U10.2 (A1); no longer U6.2 (A1)
- net RESET_5V: now also U9.10 (B2); no longer U7.12 (B2)
- net RESET_FPGA: now also U9.3 (A2); no longer U7.3 (A2)
- net RFSH_5V: now also U9.8 (B4); no longer U7.10 (B4)
- net RFSH_FPGA: now also U9.5 (A4); no longer U7.5 (A4)
- net WAIT_5V: now also U10.8 (B4); no longer U6.10 (B4)
- net WAIT_FPGA: now also U10.5 (A4); no longer U6.5 (A4)
- net WR_5V: now also U10.10 (B2); no longer U6.12 (B2)
- net WR_FPGA: now also U10.3 (A2); no longer U6.3 (A2)
- net at R2.2: now also U2.7 (OE); no longer U2.8 (OE)
- net at R10.2: now also U6.7 (OE); no longer U10.8 (OE)
- net at R9.2: now also U7.7 (OE); no longer U9.8 (OE)
- net at R4.2: now also U4.7 (OE); no longer U4.8 (OE)
- net at R7.2: now also U9.7 (OE); no longer U7.8 (OE)
- net at R6.2: now also U10.7 (OE); no longer U6.8 (OE)
- net at R5.2: now also U5.7 (OE); no longer U5.8 (OE)
- net at R8.2: now also U8.7 (OE); no longer U8.8 (OE)
- net at R1.2: now also U1.7 (OE); no longer U1.8 (OE)
- net at R3.2: now also U3.7 (OE); no longer U3.8 (OE)
