File: hardware/sip-board/peripherals.kicad_sch (KiCad schematic)
At the start: 13 parts, among them IC1 MT25QL512ABB1EW9-0SIT, J1 Conn_02x03_Odd_Even

Commit message: raahhhhh my eyeballs hurt
Other:
- moved on the sheet: R10
Changed lines of the file:
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@@
-	)
-	(junction
-		(at 109.22 152.4)
-		(diameter 0)
-		(color 0 0 0 0)
 	)
 	(junction
@@
 	)
 	(junction
+		(at 116.84 152.4)
+		(diameter 0)
+		(color 0 0 0 0)
+	)
+	(junction
 		(at 26.67 40.64)
 		(diameter 0)
@@
 	(wire
 		(pts
-			(xy 88.9 152.4) (xy 109.22 152.4)
+			(xy 88.9 152.4) (xy 116.84 152.4)
 		)
 		(stroke
@@
 	(wire
 		(pts
-			(xy 109.22 152.4) (xy 111.76 152.4)
+			(xy 116.84 152.4) (xy 119.38 152.4)
 		)
 		(stroke
@@
 	(text "https://www.tag-connect.com/wp-content/uploads/bsk-pdf-manager/2019/12/TC2030-IDC-NL-Datasheet-Rev-B.pdf"
 		(exclude_from_sim no)
-		(at 261.874 7.366 0)
+		(at 264.16 63.5 0)
 		(effects
 			(font
@@
 	(text "UG470 pg27\nNeed pull-ups on DQ2/3, CS"
 		(exclude_from_sim no)
-		(at 125.73 158.75 0)
+		(at 124.46 139.7 0)
 		(effects
 			(font
@@
 	(global_label "SPI_DQ3"
 		(shape input)
-		(at 111.76 152.4 0)
+		(at 119.38 152.4 0)
 		(fields_autoplaced yes)
 		(effects
@@
 		)
 		(property "Intersheetrefs" "${INTERSHEET_REFS}"
-			(at 123.0831 152.4 0)
+			(at 130.7031 152.4 0)
 			(effects
 				(font
@@
 	(symbol
 		(lib_id "Device:R_Small")
-		(at 109.22 154.94 180)
+		(at 116.84 154.94 180)
 		(unit 1)
 		(exclude_from_sim no)
@@
 		(fields_autoplaced yes)
 		(property "Reference" "R10"
-			(at 106.68 156.2101 0)
+			(at 114.3 156.2101 0)
 			(effects
 				(font
@@
 		)
 		(property "Value" "4k7"
-			(at 106.68 153.6701 0)
+			(at 114.3 153.6701 0)
 			(effects
 				(font
@@
 		)
 		(property "Footprint" "Resistor_SMD:R_0201_0603Metric"
-			(at 109.22 154.94 0)
+			(at 116.84 154.94 0)
 			(effects
 				(font
@@
 		)
 		(property "Datasheet" "~"
-			(at 109.22 154.94 0)
+			(at 116.84 154.94 0)
 			(effects
 				(font
@@
 		)
 		(property "Description" "Resistor, small symbol"
-			(at 109.22 154.94 0)
+			(at 116.84 154.94 0)
 			(effects
 				(font
@@
 	(symbol
 		(lib_id "power:+3V3")
-		(at 109.22 157.48 180)
+		(at 116.84 157.48 180)
 		(unit 1)
 		(exclude_from_sim no)
@@
 		(fields_autoplaced yes)
 		(property "Reference" "#PWR030"
-			(at 109.22 153.67 0)
+			(at 116.84 153.67 0)
 			(effects
 				(font
@@
 		)
 		(property "Value" "+3V3"
-			(at 109.22 162.56 0)
+			(at 116.84 162.56 0)
 			(effects
 				(font
@@
 		)
 		(property "Footprint" ""
-			(at 109.22 157.48 0)
+			(at 116.84 157.48 0)
 			(effects
 				(font
@@
 		)
 		(property "Datasheet" ""
-			(at 109.22 157.48 0)
+			(at 116.84 157.48 0)
 			(effects
 				(font
@@
 		)
 		(property "Description" "Power symbol creates a global label with name \"+3V3\""
-			(at 109.22 157.48 0)
-			(effects
-				(font
+			(at 116.84 157.48 0)
+			(effects
+				(font

Commit message: WE REDOIN PCB
Parts:
- C37: footprint Capacitor_SMD:C_0201_0603Metric -> Capacitor_SMD:C_0603_1608Metric
- C38: footprint Capacitor_SMD:C_0402_1005Metric -> Capacitor_SMD:C_0603_1608Metric
Changed lines of the file:
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@@
 			)
 		)
-		(property "Footprint" "Capacitor_SMD:C_0201_0603Metric"
+		(property "Footprint" "Capacitor_SMD:C_0603_1608Metric"
 			(at 83.82 107.95 0)
 			(effects
@@
 			)
 		)
-		(property "Footprint" "Capacitor_SMD:C_0402_1005Metric"
+		(property "Footprint" "Capacitor_SMD:C_0603_1608Metric"
 			(at 99.06 143.51 0)
 			(effects
