File: hardware/level-shifter/level-shifter.kicad_sch (KiCad schematic)
At the start: 44 parts, among them IC1 NXB0104PW-Q100J, IC10 NXB0104PW-Q100J, IC2 NXB0104PW-Q100J, IC3 NXB0104PW-Q100J, IC4 NXB0104PW-Q100J, IC5 NXB0104PW-Q100J, IC6 NXB0104PW-Q100J, IC7 NXB0104PW-Q100J, IC8 NXB0104PW-Q100J, IC9 NXB0104PW-Q100J, J1 Conn_02x24_Odd_Even, J2 Conn_01x20_Pin, J3 Conn_01x20_Pin, J4 Conn_02x24_Odd_Even

Commit message: Off for review (again)
Parts:
- C1, C10, C14, C2, C3: footprint (none) -> Capacitor_SMD:C_0805_2012Metric
- C11: renamed from C16; footprint (none) -> Capacitor_SMD:C_0805_2012Metric
- C12: renamed from C15; footprint (none) -> Capacitor_SMD:C_0805_2012Metric
- C13: renamed from C17; footprint (none) -> Capacitor_SMD:C_0805_2012Metric
- C15: renamed from C18; footprint (none) -> Capacitor_SMD:C_0805_2012Metric
- C16: renamed from C13; footprint (none) -> Capacitor_SMD:C_0805_2012Metric
- C17: renamed from C19; footprint (none) -> Capacitor_SMD:C_0805_2012Metric
- C18: renamed from C12; footprint (none) -> Capacitor_SMD:C_0805_2012Metric
- C19: renamed from C20; footprint (none) -> Capacitor_SMD:C_0805_2012Metric
- C20: renamed from C11; footprint (none) -> Capacitor_SMD:C_0805_2012Metric
- C4: renamed from C7; footprint (none) -> Capacitor_SMD:C_0805_2012Metric
- C5: renamed from C4; footprint (none) -> Capacitor_SMD:C_0805_2012Metric
- C6: renamed from C8; footprint (none) -> Capacitor_SMD:C_0805_2012Metric
- C7: renamed from C5; footprint (none) -> Capacitor_SMD:C_0805_2012Metric
- C8: renamed from C9; footprint (none) -> Capacitor_SMD:C_0805_2012Metric
- C9: renamed from C6; footprint (none) -> Capacitor_SMD:C_0805_2012Metric
Connections:
- removed net +3V3: C1.2, C12.1, C14.1, C16.1, C18.1, C20.1, C3.2, C5.2, C7.2, C9.2, IC1.1 (VCC(A)), IC10.1 (VCC(A)), IC2.1 (VCC(A)), IC3.1 (VCC(A)), IC4.1 (VCC(A)), IC5.1 (VCC(A)), IC6.1 (VCC(A)), IC7.1 (VCC(A)), IC8.1 (VCC(A)), IC9.1 (VCC(A)), J1.2 (Pin_2), J1.45 (Pin_45), J4.1 (Pin_1), J4.47 (Pin_47), J4.48 (Pin_48), R1.1, R10.1, R2.1, R3.1, R4.1, R5.1, R6.1, R7.1, R8.1, R9.1
- new net +3V3BL: C7.2, C9.2, IC4.1 (VCC(A)), IC5.1 (VCC(A)), J1.45 (Pin_45), R4.1, R5.1
- new net +3V3BR: C16.1, C18.1, C20.1, IC10.1 (VCC(A)), IC8.1 (VCC(A)), IC9.1 (VCC(A)), J4.47 (Pin_47), J4.48 (Pin_48), R10.1, R8.1, R9.1
- new net +3V3UL: C1.2, C3.2, C5.2, IC1.1 (VCC(A)), IC2.1 (VCC(A)), IC3.1 (VCC(A)), J1.2 (Pin_2), R1.1, R2.1, R3.1
- new net +3V3UR: C12.1, C14.1, IC6.1 (VCC(A)), IC7.1 (VCC(A)), J4.1 (Pin_1), R6.1, R7.1
Other:
- note added: "3.3V is broken up by quadrant to avoid current loops"
- note added: "<--- This is GND on original Z80"
- note added: "https://www.mouser.com/datasheet/2/916/NXB0104_Q100-1664477.pdf Level shifters 5V<->3V3 We are using the TSSOP-14 package OE pullup is referenced to VCC_A, >= 50k MacroFab MPNs specified"
- note removed: "This A1 --> is GND on original Z80"
- note removed: "https://www.mouser.com/datasheet/2/916/NXB0104_Q100-1664477.pdf Level shifters 5V<->3V3 We are using the XQFN12 package OE pullup is referenced to VCC_A, >= 50k MacroFab MPNs specified"
